Commit message: kuka allegro

File: gym-grabbing/gym_grabbing/envs/objects/mug/mug.urdf (robot description, URDF)
Before this commit: robot mug, 1 links, 0 joints
Links:
- link base_link: geometry collision mesh filename=mug.obj scale=0.0038 0.0038 0.0038; visual mesh filename=mug-9.obj scale=0.0038 0.0038 0.0038

File: gym-grabbing/gym_grabbing/envs/robots/baxter_description/urdf/baxter_base/baxter_base.urdf.xacro (robot description, xacro)
@@ -3,4 +3,7 @@
   <xacro:arg name="limit_scale" default="1"/>
   <xacro:arg name="gazebo" default="false"/>
+  <xacro:arg name="fixed_joints" default="{}"/>
+  <!--convert str to dict-->
+  <xacro:property name="fixed_joints_val" value="${$(arg fixed_joints)}"/>
   <xacro:if value="$(arg gazebo)">
     <!-- Gazebo Tags -->
@@ -222,6 +225,6 @@
     <child link="right_torso_itb"/>
   </joint>
-  <joint name="head_pan" type="revolute">
-    <origin rpy="0 0 0" xyz="0.06 0 0.686"/>
+  <joint name="head_pan" type="${'fixed' if 'head_pan' in fixed_joints_val else 'revolute'}">
+    <origin rpy="0 0 ${fixed_joints_val.get('head_pan', 0)}" xyz="0.06 0 0.686"/>
     <axis xyz="0 0 1"/>
     <parent link="torso"/>
@@ -519,6 +522,6 @@
     <child link="right_arm_mount"/>
   </joint>
-  <joint name="right_s0" type="revolute">
-    <origin rpy="0 0 0" xyz="0.055695 0 0.011038"/>
+  <joint name="right_s0" type="${'fixed' if 'right_s0' in fixed_joints_val else 'revolute'}">
+    <origin rpy="0 0 ${fixed_joints_val.get('right_s0', 0)}" xyz="0.055695 0 0.011038"/>
     <axis xyz="0 0 1"/>
     <parent link="right_arm_mount"/>
@@ -527,6 +530,6 @@
     <dynamics damping="0.7" friction="0.0"/>
   </joint>
-  <joint name="right_s1" type="revolute">
-    <origin rpy="-1.57079632679 0 0" xyz="0.069 0 0.27035"/>
+  <joint name="right_s1" type="${'fixed' if 'right_s1' in fixed_joints_val else 'revolute'}">
+    <origin rpy="-1.57079632679 ${fixed_joints_val.get('right_s1', 0)} 0" xyz="0.069 0 0.27035"/>
     <axis xyz="0 0 1"/>
     <parent link="right_upper_shoulder"/>
@@ -535,6 +538,6 @@
     <dynamics damping="0.7" friction="0.0"/>
   </joint>
-  <joint name="right_e0" type="revolute">
-    <origin rpy="1.57079632679 0 1.57079632679" xyz="0.102 0 0"/>
+  <joint name="right_e0" type="${'fixed' if 'right_e0' in fixed_joints_val else 'revolute'}">
+    <origin rpy="1.57079632679 ${-fixed_joints_val.get('right_e0', 0)} 1.57079632679} " xyz="0.102 0 0"/>
     <axis xyz="0 0 1"/>
     <parent link="right_lower_shoulder"/>
@@ -549,6 +552,6 @@
     <child link="right_upper_elbow_visual"/>
   </joint>
-  <joint name="right_e1" type="revolute">
-    <origin rpy="-1.57079632679 -1.57079632679 0" xyz="0.069 0 0.26242"/>
+  <joint name="right_e1" type="${'fixed' if 'right_e1' in fixed_joints_val else 'revolute'}">
+    <origin rpy="-1.57079632679 ${fixed_joints_val.get('right_e1', 0)-1.57079632679} 0" xyz="0.069 0 0.26242"/>
     <axis xyz="0 0 1"/>
     <parent link="right_upper_elbow"/>
@@ -557,6 +560,6 @@
     <dynamics damping="0.7" friction="0.0"/>
   </joint>
-  <joint name="right_w0" type="revolute">
-    <origin rpy="1.57079632679 0 1.57079632679" xyz="0.10359 0 0"/>
+  <joint name="right_w0" type="${'fixed' if 'right_w0' in fixed_joints_val else 'revolute'}">
+    <origin rpy="1.57079632679 ${-fixed_joints_val.get('right_w0', 0)} 1.57079632679" xyz="0.10359 0 0"/>
     <axis xyz="0 0 1"/>
     <parent link="right_lower_elbow"/>
@@ -577,6 +580,6 @@
     <child link="right_arm_itb"/>
   </joint>
-  <joint name="right_w1" type="revolute">
-    <origin rpy="-1.57079632679 -1.57079632679 0" xyz="0.01 0 0.2707"/>
+  <joint name="right_w1" type="${'fixed' if 'right_w1' in fixed_joints_val else 'revolute'}">
+    <origin rpy="-1.57079632679 ${fixed_joints_val.get('right_w1', 0)-1.57079632679} 0" xyz="0.01 0 0.2707"/>
     <axis xyz="0 0 1"/>
     <parent link="right_upper_forearm"/>
@@ -585,6 +588,6 @@
     <dynamics damping="0.7" friction="0.0"/>
   </joint>
-  <joint name="right_w2" type="revolute">
-    <origin rpy="1.57079632679 0 1.57079632679" xyz="0.115975 0 0"/>
+  <joint name="right_w2" type="${'fixed' if 'right_w2' in fixed_joints_val else 'revolute'}">
+    <origin rpy="1.57079632679 ${fixed_joints_val.get('right_w2', 0)} 1.57079632679" xyz="0.115975 0 0"/>
     <axis xyz="0 0 1"/>
     <parent link="right_lower_forearm"/>
@@ -887,6 +890,6 @@
     <child link="left_arm_mount"/>
   </joint>
-  <joint name="left_s0" type="revolute">
-    <origin rpy="0 0 0" xyz="0.055695 0 0.011038"/>
+  <joint name="left_s0" type="${'fixed' if 'left_s0' in fixed_joints_val else 'revolute'}">
+    <origin rpy="0 0 ${fixed_joints_val.get('left_s0', 0)}" xyz="0.055695 0 0.011038"/>
     <axis xyz="0 0 1"/>
     <parent link="left_arm_mount"/>
@@ -895,6 +898,6 @@
     <dynamics damping="0.7" friction="0.0"/>
   </joint>
-  <joint name="left_s1" type="revolute">
-    <origin rpy="-1.57079632679 0 0" xyz="0.069 0 0.27035"/>
+  <joint name="left_s1" type="${'fixed' if 'left_s1' in fixed_joints_val else 'revolute'}">
+    <origin rpy="-1.57079632679 ${fixed_joints_val.get('left_s1', 0)} 0" xyz="0.069 0 0.27035"/>
     <axis xyz="0 0 1"/>
     <parent link="left_upper_shoulder"/>
@@ -903,6 +906,6 @@
     <dynamics damping="0.7" friction="0.0"/>
   </joint>
-  <joint name="left_e0" type="revolute">
-    <origin rpy="1.57079632679 0 1.57079632679" xyz="0.102 0 0"/>
+  <joint name="left_e0" type="${'fixed' if 'left_e0' in fixed_joints_val else 'revolute'}">
+    <origin rpy="1.57079632679 ${-fixed_joints_val.get('left_e0',0)} 1.57079632679" xyz="0.102 0 0"/>
     <axis xyz="0 0 1"/>
     <parent link="left_lower_shoulder"/>
@@ -917,6 +920,6 @@
     <child link="left_upper_elbow_visual"/>
   </joint>
-  <joint name="left_e1" type="revolute">
-    <origin rpy="-1.57079632679 -1.57079632679 0" xyz="0.069 0 0.26242"/>
+  <joint name="left_e1" type="${'fixed' if 'left_e1' in fixed_joints_val else 'revolute'}">
+    <origin rpy="-1.57079632679 ${fixed_joints_val.get('left_e1', 0)-1.57079632679} 0" xyz="0.069 0 0.26242"/>
     <axis xyz="0 0 1"/>
     <parent link="left_upper_elbow"/>
@@ -925,6 +928,6 @@
     <dynamics damping="0.7" friction="0.0"/>
   </joint>
-  <joint name="left_w0" type="revolute">
-    <origin rpy="1.57079632679 0 1.57079632679" xyz="0.10359 0 0"/>
+  <joint name="left_w0" type="${'fixed' if 'left_w0' in fixed_joints_val else 'revolute'}">
+    <origin rpy="1.57079632679 ${-fixed_joints_val.get('left_w0', 0)} 1.57079632679" xyz="0.10359 0 0"/>
     <axis xyz="0 0 1"/>
     <parent link="left_lower_elbow"/>
@@ -945,6 +948,6 @@
     <child link="left_arm_itb"/>
   </joint>
-  <joint name="left_w1" type="revolute">
-    <origin rpy="-1.57079632679 -1.57079632679 0" xyz="0.01 0 0.2707"/>
+  <joint name="left_w1" type="${'fixed' if 'left_w1' in fixed_joints_val else 'revolute'}">
+    <origin rpy="-1.57079632679 ${fixed_joints_val.get('left_w1', 0)-1.57079632679} 0" xyz="0.01 0 0.2707"/>
     <axis xyz="0 0 1"/>
     <parent link="left_upper_forearm"/>
@@ -953,6 +956,6 @@
     <dynamics damping="0.7" friction="0.0"/>
   </joint>
-  <joint name="left_w2" type="revolute">
-    <origin rpy="1.57079632679 0 1.57079632679" xyz="0.115975 0 0"/>
+  <joint name="left_w2" type="${'fixed' if 'left_w2' in fixed_joints_val else 'revolute'}">
+    <origin rpy="1.57079632679 ${-fixed_joints_val.get('left_w2', 0)} 1.57079632679" xyz="0.115975 0 0"/>
     <axis xyz="0 0 1"/>
     <parent link="left_lower_forearm"/>

File: gym-grabbing/gym_grabbing/envs/robots/baxter_description/urdf/baxter_symmetric.xacro (robot description, xacro)
@@ -2,4 +2,5 @@
 <robot name="baxter" xmlns:xacro="http://www.ros.org/wiki/xacro">
   <xacro:arg name="limit_scale" default="1"/> <!--increase for higher velocities-->
+  <xacro:arg name="fixed_joints" default="{}"/>
   <xacro:arg name="gazebo" default="false"/>
   <xacro:arg name="pedestal" default="true"/>
@@ -8,4 +9,5 @@
     <xacro:arg name="gazebo" value="${gazebo}"/>
     <xacro:arg name="limit_scale" value="${limit_scale}"/>
+    <xacro:arg name="fixed_joints" value="${fixed_joints}"/>
   </xacro:include>
   <!-- Baxter Pedestal -->
@@ -32,5 +34,7 @@
                                   r_finger_tip="$(arg tip)"
                                   r_finger_grasp="$(arg grasp)"
-                                  limit_scale="$(arg limit_scale)"/>
+                                  limit_scale="$(arg limit_scale)"
+                                  fixed_joints="${$(arg fixed_joints)}"
+                                  />
   <!-- Right End Effector -->
   <!--xacro:include filename="right_end_effector.urdf.xacro" /-->
@@ -44,4 +48,6 @@
                                   r_finger_tip="$(arg tip)"
                                   r_finger_grasp="$(arg grasp)"
-                                  limit_scale="$(arg limit_scale)"/>
+                                  limit_scale="$(arg limit_scale)"
+                                  fixed_joints="${$(arg fixed_joints)}"
+                                  />
 </robot>

File: gym-grabbing/gym_grabbing/envs/robots/baxter_description/urdf/rethink_electric_gripper.xacro (robot description, xacro)
@@ -1,5 +1,5 @@
 <?xml version="1.0"?>
 <robot xmlns:xacro="http://www.ros.org/wiki/xacro" name="rethink_electric_gripper">
-  <xacro:macro name="rethink_electric_gripper" params="side r_finger r_finger_slot r_finger_tip r_finger_grasp l_finger l_finger_slot l_finger_tip l_finger_grasp limit_scale">
+  <xacro:macro name="rethink_electric_gripper" params="side r_finger r_finger_slot r_finger_tip r_finger_grasp l_finger l_finger_slot l_finger_tip l_finger_grasp limit_scale fixed_joints">
     <xacro:property name="gripper_side" value="${side[0]}" scope="local"/>
     <!-- Base of end effector -->
@@ -59,20 +59,20 @@
     <!-- Left finger -->
     <xacro:property name="l_finger_offset" value="${((l_finger_slot-1)*0.0095) -0.011}" scope="local"/>
-    <joint name="${gripper_side}_gripper_l_finger_joint" type="prismatic">
-      <origin rpy="0 0 0" xyz="0.0 ${l_finger_offset} 0.02"/>
+    <joint name="${gripper_side}_gripper_l_finger_joint" type="${'fixed' if gripper_side+'_gripper_l_finger_joint' in fixed_joints else 'prismatic'}">
+      <origin rpy="0 0 0" xyz="0.0 ${fixed_joints_val.get('head_pan', 0) + l_finger_offset} 0.02"/>
       <axis xyz="0 1 0"/>
       <parent link="${side}_gripper_base"/>
       <child link="${gripper_side}_gripper_l_finger"/>
-      <limit effort="${max(20.0*limit_scale,20.0)}" lower="0.0" upper="0.020833" velocity="${5.0*limit_scale}"/>
+      <limit effort="${max(100*limit_scale,100)}" lower="0.0" upper="0.020833" velocity="${5.0*limit_scale}"/>
       <dynamics damping="0.7" friction="0.0"/>
     </joint>
     <!-- Right finger -->
     <xacro:property name="r_finger_offset" value="${((r_finger_slot-1)*-0.0095) +0.011}" scope="local"/>
-    <joint name="${gripper_side}_gripper_r_finger_joint" type="prismatic">
-      <origin rpy="0 0 0" xyz="0.0 ${r_finger_offset} 0.02"/>
+    <joint name="${gripper_side}_gripper_r_finger_joint" type="${'fixed' if gripper_side+'_gripper_r_finger_joint' in fixed_joints else 'prismatic'}">
+      <origin rpy="0 0 0" xyz="0.0 ${fixed_joints_val.get('head_pan', 0) + r_finger_offset} 0.02"/>
       <axis xyz="0 1 0"/>
       <parent link="${side}_gripper_base"/>
       <child link="${gripper_side}_gripper_r_finger"/>
-      <limit effort="${max(20.0*limit_scale,20.0)}" lower="-0.020833" upper="0.0" velocity="${5.0*limit_scale}"/>
+      <limit effort="${max(100*limit_scale,100)}" lower="-0.020833" upper="0.0" velocity="${5.0*limit_scale}"/>
       <mimic joint="${gripper_side}_gripper_l_finger_joint" multiplier="-1.0"/>
       <dynamics damping="0.7" friction="0.0"/>
