Commit message: quality energy

File: gym-grabbing/gym_grabbing/envs/robots/LBR_iiwa/urdf/lbr_iiwa_14_r820_macro.xacro (robot description, xacro)
@@ -188,5 +188,5 @@
       <child link="${prefix}link_1" />
       <axis xyz="0 0 1" />
-      <limit lower="-2.9668" upper="2.9668" effort="50" velocity="1.4834" />
+      <limit lower="-2.9668" upper="2.9668" effort="176" velocity="1.4834" />
     </joint>
     <joint name="${prefix}joint_a2" type="revolute">
@@ -195,5 +195,5 @@
       <child link="${prefix}link_2" />
       <axis xyz="0 1 0" />
-      <limit lower="-2.0942" upper="2.0942" effort="100" velocity="1.4834" />
+      <limit lower="-2.0942" upper="2.0942" effort="176" velocity="1.4834" />
     </joint>
     <joint name="${prefix}joint_a3" type="revolute">
@@ -202,5 +202,5 @@
       <child link="${prefix}link_3" />
       <axis xyz="0 0 1" />
-      <limit lower="-2.9668" upper="2.9668" effort="50" velocity="1.7452" />
+      <limit lower="-2.9668" upper="2.9668" effort="110" velocity="1.7452" />
     </joint>
     <joint name="${prefix}joint_a4" type="revolute">
@@ -209,5 +209,5 @@
       <child link="${prefix}link_4" />
       <axis xyz="0 -1 0" />
-      <limit lower="-2.0942" upper="2.0942" effort="50" velocity="1.3089" />
+      <limit lower="-2.0942" upper="2.0942" effort="110" velocity="1.3089" />
     </joint>
     <joint name="${prefix}joint_a5" type="revolute">
@@ -216,5 +216,5 @@
       <child link="${prefix}link_5" />
       <axis xyz="0 0 1" />
-      <limit lower="-2.9668" upper="2.9668" effort="50" velocity="2.2688" />
+      <limit lower="-2.9668" upper="2.9668" effort="110" velocity="2.2688" />
     </joint>
     <joint name="${prefix}joint_a6" type="revolute">
@@ -223,5 +223,5 @@
       <child link="${prefix}link_6" />
       <axis xyz="0 1 0" />
-      <limit lower="-2.0942" upper="2.0942" effort="50" velocity="2.356" />
+      <limit lower="-2.0942" upper="2.0942" effort="40" velocity="2.356" />
     </joint>
     <joint name="${prefix}joint_a7" type="revolute">
@@ -230,5 +230,5 @@
       <child link="${prefix}link_7" />
       <axis xyz="0 0 1" />
-      <limit lower="-3.0541" upper="3.0541" effort="10" velocity="2.356" />
+      <limit lower="-3.0541" upper="3.0541" effort="40" velocity="2.356" />
     </joint>
     <joint name="${prefix}joint_a7-end_effector" type="fixed">

File: gym-grabbing/gym_grabbing/envs/robots/LBR_iiwa/urdf/lbr_iiwa_robotiq.xacro (robot description, xacro)
@@ -20,3 +20,31 @@
     <child link="robotiq_arg2f_base_link"/>
   </joint>
+  <link name="base">
+      <inertial>
+        <origin rpy="0 0 0" xyz="0 0 0"/>
+        <mass value="10"/>
+        <inertia ixx="1" ixy="0" ixz="0" iyy="1" iyz="0" izz="1"/>
+      </inertial>
+    <visual>
+      <origin xyz="0 0 0" rpy="0 0 0" />
+      <geometry>
+          <box size=" 1 2 0.5 "/>
+      </geometry>
+      <material name="Grey"/>
+    </visual>
+    <collision>
+      <origin xyz="0 0 0" rpy="0 0 0" />
+      <geometry>
+          <box size=" 0.5 0.5 0.5 "/>
+      </geometry>
+    </collision>
+    <contact>
+        <lateral_friction value="0.1"/>
+    </contact>
+  </link>
+  <joint name="base_to_kuka" type="fixed">
+    <origin xyz="0 0 0.25" rpy="0 0 0"/>
+    <parent link="base"/>
+    <child link="kuka_base_link"/>
+  </joint>
 </robot>

File: gym-grabbing/gym_grabbing/envs/robots/robotiq_140_gripper_description/urdf/robotiq_140.urdf.xacro (robot description, xacro)
@@ -143,14 +143,26 @@
           <mesh filename="package://robotiq_140_gripper_description/meshes/robotiq_140_left_inner_finger.dae" scale="0.001 0.001 0.001" />
         </geometry>
-        <material name="Gazebo/Black">
-          <color rgba="0.1 0.1 0.1 1" />
-        </material>
-      </visual>
-      <collision>
-        <origin xyz="0 0 0" rpy="0 0 0" />
-        <geometry>
-          <mesh filename="package://robotiq_140_gripper_description/meshes/robotiq_140_left_inner_finger.obj" scale="0.001 0.001 0.001" />
-        </geometry>
-      </collision>
+        <!--origin xyz="-0.022 0 0.046" rpy="0 0 0" />
+        <geometry>
+            <box size=" 0.0064 0.022 0.065 "></box>
+        </geometry-->
+        <material name="Gazebo/Black">
+          <color rgba="0.1 0.1 0.1 1" />
+        </material>
+      </visual>
+      <collision>
+        <origin xyz="0 0 0" rpy="0 0 0" />
+        <geometry>
+          <mesh filename="package://robotiq_140_gripper_description/meshes/robotiq_140_left_inner_finger.dae" scale="0.001 0.001 0.001" />
+        </geometry>
+        <!--origin xyz="-0.022 0 0.046" rpy="0 0 0" />
+        <geometry>
+            <box size=" 0.0064 0.022 0.065 "></box>
+        </geometry-->
+      </collision>
+      <!--contact>
+          <rolling_friction value="0.01"/>
+          <spinning_friction value="0.01"/>
+      </contact-->
     </link>
     <gazebo reference="${prefix}left_inner_finger">
@@ -169,12 +181,16 @@
           <mesh filename="package://robotiq_140_gripper_description/meshes/robotiq_140_right_inner_finger.dae" scale="0.001 0.001 0.001"/>
         </geometry>
-        <material name="Gazebo/Black">
-          <color rgba="0.1 0.1 0.1 1" />
-        </material>
-      </visual>
-      <collision>
-        <origin xyz="0 0 0" rpy="0 0 0" />
-        <geometry>
-          <mesh filename="package://robotiq_140_gripper_description/meshes/robotiq_140_right_inner_finger.obj" scale="0.001 0.001 0.001"/>
+        <!--origin xyz="0.022 0 0.046" rpy="0 0 0" />
+        <geometry>
+            <box size=" 0.0064 0.022 0.065 "></box>
+        </geometry-->
+        <material name="Gazebo/Black">
+          <color rgba="0.1 0.1 0.1 1" />
+        </material>
+      </visual>
+      <collision>
+        <origin xyz="0 0 0" rpy="0 0 0" />
+        <geometry>
+          <mesh filename="package://robotiq_140_gripper_description/meshes/robotiq_140_right_inner_finger.dae" scale="0.001 0.001 0.001"/>
         </geometry>
       </collision>
